File: tigard.kicad_pcb (KiCad board)
At the start: 4 copper layers, 46 x 46 mm, 92 parts, among them J1 USB_C_Receptacle_USB2.0, J2 JTAG, J3 UART, J4 SPI, J5 CORTEX, J6 LA, J7 I2C, Q1 BSH103, SW1 TARGET, SW2 MODE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

Commit message: v3.1
Parts:
- removed J5: CORTEX, tigard:PinHeader_2x05_P1.27mm_Vertical_SMD
- removed J6: LA, tigard:PinHeader_2x07_P1.27mm_Vertical_SMD
- added J8: CORTEX, mybays_connector:debugger_2x05_P1.27mm_Vertical, F.Cu at (71.8, 41.3)
- added J9: LA, Connector_PinHeader_1.27mm:PinHeader_2x07_P1.27mm_Vertical, F.Cu at (52.8, 69.9)
Connections:
- J1 pad A8: (no net) -> Net-(J1-PadA8)
- J1 pad B8: (no net) -> Net-(J1-PadB8)
- RN6 pad 3: (no net) -> Net-(RN6-Pad3)
- RN6 pad 4: (no net) -> Net-(RN6-Pad4)
- SW1 pad 1: (no net) -> Net-(SW1-Pad1)
- SW1 pad 2: (no net) -> Net-(SW1-Pad2)
- SW1 pad 3: (no net) -> Net-(SW1-Pad3)
- SW1 pad 4: (no net) -> Net-(SW1-Pad4)
- SW1 pad 5: (no net) -> Net-(SW1-Pad5)
- U1 pad 4: (no net) -> Net-(U1-Pad4)
- U2 pad 4: (no net) -> Net-(U2-Pad4)
- U3 pad 24: (no net) -> Net-(U3-Pad24)
- U3 pad 26: (no net) -> Net-(U3-Pad26)
- U3 pad 27: (no net) -> Net-(U3-Pad27)
- U3 pad 28: (no net) -> Net-(U3-Pad28)
- U3 pad 32: (no net) -> Net-(U3-Pad32)
- U3 pad 33: (no net) -> Net-(U3-Pad33)
- U3 pad 34: (no net) -> Net-(U3-Pad34)
- U3 pad 36: (no net) -> Net-(U3-Pad36)
- U3 pad 48: (no net) -> Net-(U3-Pad48)
- U3 pad 52: (no net) -> Net-(U3-Pad52)
- U3 pad 53: (no net) -> Net-(U3-Pad53)
- U3 pad 54: (no net) -> Net-(U3-Pad54)
- U3 pad 55: (no net) -> Net-(U3-Pad55)
- U3 pad 57: (no net) -> Net-(U3-Pad57)
- U3 pad 58: (no net) -> Net-(U3-Pad58)
- U3 pad 59: (no net) -> Net-(U3-Pad59)
Routing:
- net GND: track 50.4 -> 56.0 mm
- net /xPB4: track 37.9 -> 43.0 mm
- net /ICE_CDONE: track 74.9 -> 80.0 mm
- net /DI: track 56.2 -> 52.5 mm, vias 3 -> 2
- net /xPB5: track 64.2 -> 60.7 mm, vias 2 -> 0
- net /CS: track 66.3 -> 63.3 mm, vias 2 -> 1
- net /UART_TX: track 63.0 -> 61.2 mm, vias 2 -> 1
- net /CIPO: track 64.5 -> 62.7 mm, vias 1 -> 2
- net VTARGET: track 129.2 -> 130.6 mm
- net /COPI: track 104.5 -> 105.7 mm, vias 3 -> 2
- net /CLK: track 87.3 -> 87.9 mm, vias 3 -> 1
- net /CORTEX_PIN2: track 12.7 -> 12.4 mm, vias 1 -> 0
