File: tigard.sch (KiCad schematic (older format))
At the start: 93 parts, among them J1 USB_C_Receptacle_USB2.0, J2 JTAG, J3 UART, J4 SPI, J5 CORTEX, J6 LA, J7 I2C, J8 CORTEX, J9 LA, Q1 BSH103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

Commit message: v.2.2
Parts:
- removed J8: CORTEX, mybays_connector:debugger_2x05_P1.27mm_Vertical, symbol Connector_Generic:Conn_02x05_Odd_Even
- removed J9: LA, Connector_PinHeader_1.27mm:PinHeader_2x07_P1.27mm_Vertical, symbol Connector_Generic:Conn_02x07_Odd_Even
Connections:
- no-connect marks 35 -> 30
Changed lines of the file:
@@
 Wire Wire Line
 	2600 4100 2600 4150
-$Comp
-L Connector_Generic:Conn_02x05_Odd_Even J8
-U 1 1 606E7698
-P 13200 2300
-F 0 "J8" H 13250 2717 50  0000 C CNN
-F 1 "CORTEX" H 13250 2626 50  0000 C CNN
-F 2 "mybays_connector:debugger_2x05_P1.27mm_Vertical" H 13200 2300 50  0001 C CNN
-F 3 "~" H 13200 2300 50  0001 C CNN
-F 4 "FTSH-105-01-F-DV-K" H 13200 2300 50  0001 C CNN "P/N"
-F 5 "C448647" H 13200 2300 50  0001 C CNN "LCSC"
-F 6 "conn-th-01in-5-2-hdr" H 13200 2300 50  0001 C CNN "Key"
-	1    13200 2300
-	1    0    0    -1
-$EndComp
-NoConn ~ 13000 2400
-Text Label 14000 2500 2    50   ~ 0
-~SRST
-$Comp
-L power:GND #PWR0163
-U 1 1 606E76A0
-P 12850 2550
-F 0 "#PWR0163" H 12850 2300 50  0001 C CNN
-F 1 "GND" H 12855 2377 50  0000 C CNN
-F 2 "" H 12850 2550 50  0001 C CNN
-F 3 "" H 12850 2550 50  0001 C CNN
-	1    12850 2550
-	1    0    0    -1
-$EndComp
-Wire Wire Line
-	12850 2200 13000 2200
-Wire Wire Line
-	13000 2300 12850 2300
-Connection ~ 12850 2300
-Wire Wire Line
-	12850 2300 12850 2200
-Wire Wire Line
-	12850 2300 12850 2500
-Wire Wire Line
-	12850 2500 13000 2500
-Connection ~ 12850 2500
-Wire Wire Line
-	12850 2500 12850 2550
-Text Label 14000 2200 2    50   ~ 0
-TCK
-Text Label 14000 2100 2    50   ~ 0
-CORTEX_PIN2
-Text Label 14000 2300 2    50   ~ 0
-TDO
-Text Label 14000 2400 2    50   ~ 0
-TDI
-Wire Wire Line
-	13500 2100 14000 2100
-Wire Wire Line
-	13500 2200 14000 2200
-Wire Wire Line
-	13500 2300 14000 2300
-Wire Wire Line
-	13500 2400 14000 2400
-Wire Wire Line
-	13500 2500 14000 2500
-$Comp
-L tigard:VTARGET #PWR0164
-U 1 1 606E76B7
-P 12850 2050
-F 0 "#PWR0164" H 12850 1900 50  0001 C CNN
-F 1 "VTARGET" H 12865 2223 50  0000 C CNN
-F 2 "" H 12850 2050 50  0001 C CNN
-F 3 "" H 12850 2050 50  0001 C CNN
-	1    12850 2050
-	1    0    0    -1
-$EndComp
-Wire Wire Line
-	12850 2050 12850 2100
-Wire Wire Line
-	12850 2100 13000 2100
-$Comp
-L Connector_Generic:Conn_02x07_Odd_Even J9
-U 1 1 607DD367
-P 13350 3600
-F 0 "J9" H 13400 4117 50  0000 C CNN
-F 1 "LA" H 13400 4026 50  0000 C CNN
-F 2 "Connector_PinHeader_1.27mm:PinHeader_2x07_P1.27mm_Vertical" H 13350 3600 50  0001 C CNN
-F 3 "~" H 13350 3600 50  0001 C CNN
-F 4 "FTSH-107-01-F-DV-K" H 13350 3600 50  0001 C CNN "P/N"
-F 5 "" H 13350 3600 50  0001 C CNN "LCSC"
-	1    13350 3600
-	1    0    0    -1
-$EndComp
-NoConn ~ 13150 3800
-NoConn ~ 13150 3900
-NoConn ~ 13650 3900
-NoConn ~ 13650 3800
-Text Label 12900 3300 0    50   ~ 0
-xPB0
-Text Label 12900 3400 0    50   ~ 0
-xPB2
-Text Label 12900 3500 0    50   ~ 0
-xPB4
-Text Label 12900 3600 0    50   ~ 0
-xPB6
-Text Label 13900 3300 2    50   ~ 0
-xPB1
-Text Label 13900 3400 2    50   ~ 0
-xPB3
-Text Label 13900 3500 2    50   ~ 0
-xPB5
-Text Label 13900 3600 2    50   ~ 0
-xPB7
-Wire Wire Line
-	13900 3600 13650 3600
-Wire Wire Line
-	13900 3500 13650 3500
-Wire Wire Line
-	13650 3400 13900 3400
-Wire Wire Line
-	13900 3300 13650 3300
-Wire Wire Line
-	13150 3300 12900 3300
-Wire Wire Line
-	12900 3400 13150 3400
-Wire Wire Line
-	13150 3500 12900 3500
-Wire Wire Line
-	12900 3600 13150 3600
-$Comp
-L power:GND #PWR0165
-U 1 1 607DD381
-P 13750 4050
-F 0 "#PWR0165" H 13750 3800 50  0001 C CNN
-F 1 "GND" H 13755 3877 50  0000 C CNN
-F 2 "" H 13750 4050 50  0001 C CNN
-F 3 "" H 13750 4050 50  0001 C CNN
-	1    13750 4050
-	1    0    0    -1
-$EndComp
-Wire Wire Line
-	13650 3700 13750 3700
-Wire Wire Line
-	13750 3700 13750 4000
-Wire Wire Line
-	13150 3700 13050 3700
-Wire Wire Line
-	13050 3700 13050 4000
-Wire Wire Line
-	13050 4000 13750 4000
-Connection ~ 13750 4000
-Wire Wire Line
-	13750 4000 13750 4050
 $EndSCHEMATC

Commit message: v3.1
Parts:
- removed J5: CORTEX, tigard:PinHeader_2x05_P1.27mm_Vertical_SMD, symbol Connector_Generic:Conn_02x05_Odd_Even
- removed J6: LA, tigard:PinHeader_2x07_P1.27mm_Vertical_SMD, symbol Connector_Generic:Conn_02x07_Odd_Even
- added CON1: CORTEX-DEBUGGER_HOST, mybays_connector:debugger_2x05_P1.27mm_Vertical, symbol mybays_connector:CORTEX-DEBUGGER_HOST
- added J8: CORTEX, mybays_connector:debugger_2x05_P1.27mm_Vertical, symbol Connector_Generic:Conn_02x05_Odd_Even
- added J9: LA, Connector_PinHeader_1.27mm:PinHeader_2x07_P1.27mm_Vertical, symbol Connector_Generic:Conn_02x07_Odd_Even
Connections:
- net CIPO: now also J8.6 (Pin_6)
- net CLK: now also J8.4 (Pin_4), J9.1 (Pin_1)
- net COPI: now also J8.8 (Pin_8), J9.2 (Pin_2)
- net CORTEX_PIN2: now also J8.2 (Pin_2)
- net CS: now also J9.4 (Pin_4)
- net DI: now also J9.3 (Pin_3)
- net GND: now also CON1.6 (GND), CON1.9 (GND), J8.3 (Pin_3), J8.5 (Pin_5), J8.9 (Pin_9), J9.10 (Pin_10), J9.9 (Pin_9)
- net ICE_CDONE: now also CON1.10 (RXD), J9.8 (Pin_8)
- net UART_TX: now also CON1.8 (TXD), J9.7 (Pin_7)
- net VTARGET: now also CON1.3 (3.3V), J8.1 (Pin_1)
- net xPB4: now also J9.5 (Pin_5)
- net xPB5: now also CON1.2 (RST), J8.10 (Pin_10), J9.6 (Pin_6)
